Commit message: improved urdf with mesh and macros

File: urdf/robot_arms.xacro (robot description, xacro)
@@ -1,6 +1,31 @@
 <?xml version="1.0"?>
 <robot xmlns:xacro="http://www.ros.org/wiki/xacro" >
-    <xacro:property name="short_arm_length" value="0.050"/>
+    <xacro:property name="short_arm_length" value="0.075"/>
     <xacro:property name="long_arm_length" value="0.133"/>
+    <xacro:macro name="short_arm_link" params="link_name">
+        <link name="${link_name}">
+            <visual>
+                <material name="white"/>
+                <geometry>
+                    <cylinder length = "${short_arm_length}" radius = "0.005"/>
+                </geometry>
+                <origin xyz="0 ${short_arm_length / 2 } 0" rpy="1.5708 0 0"/>
+            </visual>
+            <collision>
+                <geometry>
+                    <cylinder length = "${short_arm_length}" radius = "0.005"/>
+                </geometry>
+                <origin xyz="0 ${short_arm_length / 2 } 0" rpy="1.5708 0 0"/>
+            </collision>
+            <inertial>
+                <origin xyz="0 ${short_arm_length / 2 } 0" rpy="1.5708 0 0"/>
+                <mass value="0.060"/>
+                <inertia
+                    ixx="0.00001" ixy="0.0" ixz="0.0"
+                    iyy="0.0000065" iyz="0.0"
+                    izz="0.0000125"/>
+            </inertial>
+        </link>
+    </xacro:macro>
     <joint name="short_arm1_joint" type="revolute">
         <parent link="servo1_link"/>
@@ -10,12 +35,5 @@
         <limit lower="-1.5708" upper="1.5708" effort="100" velocity="100"/>
     </joint>
-    <link name="short_arm1_link">
-        <visual>
-            <geometry>
-                <cylinder length = "${short_arm_length}" radius = "0.005"/>
-            </geometry>
-            <origin xyz="0 ${short_arm_length / 2 } 0" rpy="1.5708 0 0"/>
-        </visual>
-    </link>
+    <xacro:short_arm_link link_name="short_arm1_link"/>
     <joint name="short_arm2_joint" type="revolute">
         <parent link="servo2_link"/>
@@ -25,12 +43,5 @@
         <limit lower="-1.5708" upper="1.5708" effort="100" velocity="100"/>
     </joint>
-    <link name="short_arm2_link">
-        <visual>
-            <geometry>
-                <cylinder length = "${short_arm_length}" radius = "0.005"/>
-            </geometry>
-            <origin xyz="0 ${short_arm_length / 2 } 0" rpy="1.5708 0 0"/>
-        </visual>
-    </link>
+    <xacro:short_arm_link link_name="short_arm2_link"/>
     <joint name="short_arm3_joint" type="revolute">
         <parent link="servo3_link"/>
@@ -40,12 +51,5 @@
         <limit lower="-1.5708" upper="1.5708" effort="100" velocity="100"/>
     </joint>
-    <link name="short_arm3_link">
-        <visual>
-            <geometry>
-                <cylinder length = "${short_arm_length}" radius = "0.005"/>
-            </geometry>
-            <origin xyz="0 ${short_arm_length / 2 } 0" rpy="1.5708 0 0"/>
-        </visual>
-    </link>
+    <xacro:short_arm_link link_name="short_arm3_link"/>
     <joint name="short_arm4_joint" type="revolute">
         <parent link="servo4_link"/>
@@ -55,12 +59,5 @@
         <limit lower="-1.5708" upper="1.5708" effort="100" velocity="100"/>
     </joint>
-    <link name="short_arm4_link">
-        <visual>
-            <geometry>
-                <cylinder length = "${short_arm_length}" radius = "0.005"/>
-            </geometry>
-            <origin xyz="0 ${short_arm_length / 2 } 0" rpy="1.5708 0 0"/>
-        </visual>
-    </link>
+    <xacro:short_arm_link link_name="short_arm4_link"/>
     <joint name="short_arm5_joint" type="revolute">
         <parent link="servo5_link"/>
@@ -70,12 +67,5 @@
         <limit lower="-1.5708" upper="1.5708" effort="100" velocity="100"/>
     </joint>
-    <link name="short_arm5_link">
-        <visual>
-            <geometry>
-                <cylinder length = "${short_arm_length}" radius = "0.005"/>
-            </geometry>
-            <origin xyz="0 ${short_arm_length / 2 } 0" rpy="1.5708 0 0"/>
-        </visual>
-    </link>
+    <xacro:short_arm_link link_name="short_arm5_link"/>
     <joint name="short_arm6_joint" type="revolute">
         <parent link="servo6_link"/>
@@ -85,11 +75,4 @@
         <limit lower="-1.5708" upper="1.5708" effort="100" velocity="100"/>
     </joint>
-    <link name="short_arm6_link">
-        <visual>
-            <geometry>
-                <cylinder length = "${short_arm_length}" radius = "0.005"/>
-            </geometry>
-            <origin xyz="0 ${short_arm_length / 2 } 0" rpy="1.5708 0 0"/>
-        </visual>
-    </link>
+    <xacro:short_arm_link link_name="short_arm6_link"/>
 </robot>

File: urdf/robot_base.xacro (robot description, xacro)
@@ -19,23 +19,57 @@
     <xacro:property name="servo6_y" value="-0.0525"/>
     <material name="white">
-        <color rgba="1 1 1 1"/>
+        <color rgba="0.95 0.95 0.95 1"/>
     </material>
     <material name="black">
-        <color rgba="0 0 0 1"/>
+        <color rgba="0.2 0.2 0.2 1"/>
     </material>
-    <link name="world"/>
-    <joint name="base_joint" type="fixed">
-        <parent link="world"/>
-        <child link="base_link"/>
-        <origin xyz="0 0 0"/>
-    </joint>
     <link name="base_link">
         <visual>
+            <material name="white"/>
+            <geometry>
+                <mesh filename="package://robot/urdf/simplified_base_model.stl"/>
+            </geometry>
+            <origin xyz="0 0 0" rpy="0 0 -0.523"/>
+        </visual>
+        <collision>
             <geometry>
                 <cylinder length = "0.04" radius = "0.06"/>
             </geometry>
             <origin xyz="0 0 0.02"/>
-        </visual>
+        </collision>
+        <inertial>
+            <origin xyz="0 0 1" rpy="0 0 0"/>
+            <mass value="0.15"/>
+            <inertia
+                ixx="0.00024" ixy="0.0" ixz="0.0"
+                iyy="0.00025" iyz="0.0"
+                izz="0.00041"/>
+        </inertial>
     </link>
+    <xacro:macro name="servo_link" params="link_name">
+        <link name="${link_name}">
+            <visual>
+                <material name="black"/>
+                <geometry>
+                    <box size="0.030 0.040 0.020"/>
+                </geometry>
+                <origin xyz="-0.023 -0.010 0"/>
+            </visual>
+            <collision>
+                <geometry>
+                    <box size="0.030 0.040 0.020"/>
+                </geometry>
+                <origin xyz="-0.023 -0.010 0"/>
+            </collision>
+            <inertial>
+                <origin xyz="-0.023 -0.010 0"/>
+                <mass value="0.060"/>
+                <inertia
+                    ixx="0.00001" ixy="0.0" ixz="0.0"
+                    iyy="0.0000065" iyz="0.0"
+                    izz="0.0000125"/>
+            </inertial>
+        </link>
+    </xacro:macro>
     <joint name="servo1_joint" type="fixed">
         <parent link="base_link"/>
@@ -43,12 +77,5 @@
         <origin xyz="${servo1_x} ${servo1_y} ${servo_height}" rpy="0 ${draft_angle} ${_120_degrees}"/>
     </joint>
-    <link name="servo1_link">
-        <visual>
-            <geometry>
-                <box size="0.030 0.040 0.020"/>
-            </geometry>
-            <origin xyz="-0.023 -0.010 0"/>
-        </visual>
-    </link>
+    <xacro:servo_link link_name="servo1_link"/>
     <joint name="servo2_joint" type="fixed">
         <parent link="base_link"/>
@@ -56,12 +83,5 @@
         <origin xyz="${servo2_x} ${servo2_y} ${servo_height}" rpy="${_180_degrees} ${draft_angle} ${_120_degrees}"/>
     </joint>
-    <link name="servo2_link">
-        <visual>
-            <geometry>
-                <box size="0.030 0.040 0.020"/>
-            </geometry>
-            <origin xyz="-0.023 -0.010 0"/>
-        </visual>
-    </link>
+    <xacro:servo_link link_name="servo2_link"/>
     <joint name="servo3_joint" type="fixed">
         <parent link="base_link"/>
@@ -69,12 +89,5 @@
         <origin xyz="${servo3_x} ${servo3_y} ${servo_height}" rpy="0 ${draft_angle} 0"/>
     </joint>
-    <link name="servo3_link">
-        <visual>
-            <geometry>
-                <box size="0.030 0.040 0.020"/>
-            </geometry>
-            <origin xyz="-0.023 -0.010 0"/>
-        </visual>
-    </link>
+    <xacro:servo_link link_name="servo3_link"/>
     <joint name="servo4_joint" type="fixed">
         <parent link="base_link"/>
@@ -82,12 +95,5 @@
         <origin xyz="${servo4_x} ${servo4_y} ${servo_height}" rpy="${_180_degrees} ${draft_angle} 0"/>
     </joint>
-    <link name="servo4_link">
-        <visual>
-            <geometry>
-                <box size="0.030 0.040 0.020"/>
-            </geometry>
-            <origin xyz="-0.023 -0.010 0"/>
-        </visual>
-    </link>
+    <xacro:servo_link link_name="servo4_link"/>
     <joint name="servo5_joint" type="fixed">
         <parent link="base_link"/>
@@ -95,12 +101,5 @@
         <origin xyz="${servo5_x} ${servo5_y} ${servo_height}" rpy="0 ${draft_angle} ${_240_degrees}"/>
     </joint>
-    <link name="servo5_link">
-        <visual>
-            <geometry>
-                <box size="0.030 0.040 0.020"/>
-            </geometry>
-            <origin xyz="-0.023 -0.010 0"/>
-        </visual>
-    </link>
+    <xacro:servo_link link_name="servo5_link"/>
     <joint name="servo6_joint" type="fixed">
         <parent link="base_link"/>
@@ -108,11 +107,4 @@
         <origin xyz="${servo6_x} ${servo6_y} ${servo_height}" rpy="${_180_degrees} ${draft_angle} ${_240_degrees}"/>
     </joint>
-    <link name="servo6_link">
-        <visual>
-            <geometry>
-                <box size="0.030 0.040 0.020"/>
-            </geometry>
-            <origin xyz="-0.023 -0.010 0"/>
-        </visual>
-    </link>
+    <xacro:servo_link link_name="servo6_link"/>
 </robot>
