Commit message: simulation kinda working

File: urdf/robot.urdf.xacro (robot description, xacro)
@@ -3,3 +3,4 @@
     <xacro:include filename="robot_base.xacro" />
     <xacro:include filename="robot_arms.xacro" />
+    <xacro:include filename="robot_gazebo.xacro" />
 </robot>

File: urdf/robot_arms.xacro (robot description, xacro)
@@ -2,5 +2,5 @@
 <robot xmlns:xacro="http://www.ros.org/wiki/xacro" >
     <xacro:property name="short_arm_length" value="0.075"/>
-    <xacro:property name="long_arm_length" value="0.133"/>
+    <xacro:property name="long_arm_length" value="0.190"/>
     <xacro:macro name="short_arm_link" params="link_name">
         <link name="${link_name}">
@@ -34,4 +34,5 @@
         <axis xyz="1 0 0"/>
         <limit lower="-1.5708" upper="1.5708" effort="100" velocity="100"/>
+        <dynamics damping="10.0" friction="10.0"/>
     </joint>
     <xacro:short_arm_link link_name="short_arm1_link"/>
@@ -42,4 +43,5 @@
         <axis xyz="1 0 0"/>
         <limit lower="-1.5708" upper="1.5708" effort="100" velocity="100"/>
+        <dynamics damping="10.0" friction="10.0"/>
     </joint>
     <xacro:short_arm_link link_name="short_arm2_link"/>
@@ -50,4 +52,5 @@
         <axis xyz="1 0 0"/>
         <limit lower="-1.5708" upper="1.5708" effort="100" velocity="100"/>
+        <dynamics damping="10.0" friction="10.0"/>
     </joint>
     <xacro:short_arm_link link_name="short_arm3_link"/>
@@ -58,4 +61,5 @@
         <axis xyz="1 0 0"/>
         <limit lower="-1.5708" upper="1.5708" effort="100" velocity="100"/>
+        <dynamics damping="10.0" friction="10.0"/>
     </joint>
     <xacro:short_arm_link link_name="short_arm4_link"/>
@@ -66,4 +70,5 @@
         <axis xyz="1 0 0"/>
         <limit lower="-1.5708" upper="1.5708" effort="100" velocity="100"/>
+        <dynamics damping="10.0" friction="10.0"/>
     </joint>
     <xacro:short_arm_link link_name="short_arm5_link"/>
@@ -74,4 +79,5 @@
         <axis xyz="1 0 0"/>
         <limit lower="-1.5708" upper="1.5708" effort="100" velocity="100"/>
+        <dynamics damping="10.0" friction="10.0"/>
     </joint>
     <xacro:short_arm_link link_name="short_arm6_link"/>

File: urdf/robot_base.xacro (robot description, xacro)
@@ -28,7 +28,8 @@
             <material name="white"/>
             <geometry>
-                <mesh filename="package://robot/urdf/simplified_base_model.stl"/>
+                <cylinder length = "0.04" radius = "0.06"/>
+                <!-- <mesh filename="package://robot/urdf/simplified_base_model.stl"/> -->
             </geometry>
-            <origin xyz="0 0 0" rpy="0 0 -0.523"/>
+            <origin xyz="0 0 0.02" rpy="0 0 -0.523"/>
         </visual>
         <collision>
