Commit message: mass commit

File: urdf/robot.urdf (robot description, URDF)
Before this commit: robot robot, 13 links, 12 joints
Links:
- added link collision_link1, mass 0.06; collision sphere radius=0.02; visual sphere radius=0.02
- added link collision_link2, mass 0.06; collision sphere radius=0.02; visual sphere radius=0.02
- added link collision_link3, mass 0.06; collision sphere radius=0.02; visual sphere radius=0.02
- added link end_short_arm1_link, mass 0.01; collision sphere radius=0.0075; visual sphere radius=0.0075
- added link end_short_arm2_link, mass 0.01; collision sphere radius=0.0075; visual sphere radius=0.0075
- added link end_short_arm3_link, mass 0.01; collision sphere radius=0.0075; visual sphere radius=0.0075
- added link end_short_arm4_link, mass 0.01; collision sphere radius=0.0075; visual sphere radius=0.0075
- added link end_short_arm5_link, mass 0.01; collision sphere radius=0.0075; visual sphere radius=0.0075
- added link end_short_arm6_link, mass 0.01; collision sphere radius=0.0075; visual sphere radius=0.0075
- link base_link: geometry visual cylinder length=0.035 radius=0.06
- link servo1_link: geometry visual box size=0.030 0.040 0.020
- link servo2_link: geometry visual box size=0.030 0.040 0.020
- link servo3_link: geometry visual box size=0.030 0.040 0.020
- link servo4_link: geometry visual box size=0.030 0.040 0.020
- link servo5_link: geometry visual box size=0.030 0.040 0.020
- link servo6_link: geometry visual box size=0.030 0.040 0.020
- link short_arm1_link: geometry visual cylinder length=0.075 radius=0.005
- link short_arm2_link: geometry visual cylinder length=0.075 radius=0.005
- link short_arm3_link: geometry visual cylinder length=0.075 radius=0.005
- link short_arm4_link: geometry visual cylinder length=0.075 radius=0.005
- link short_arm5_link: geometry visual cylinder length=0.075 radius=0.005
- link short_arm6_link: geometry visual cylinder length=0.075 radius=0.005
Joints:
- added joint collision_joint1: type fixed, parent base_link, child collision_link1, origin xyz=-0.06 0.0 0.02
- added joint collision_joint2: type fixed, parent base_link, child collision_link2, origin xyz=0.03 -0.0519 0.02
- added joint collision_joint3: type fixed, parent base_link, child collision_link3, origin xyz=0.03 0.0519 0.02
- added joint end_short_arm1_joint: type fixed, parent short_arm1_link, child end_short_arm1_link, origin xyz=0 0.075 0
- added joint end_short_arm2_joint: type fixed, parent short_arm2_link, child end_short_arm2_link, origin xyz=0 0.075 0
- added joint end_short_arm3_joint: type fixed, parent short_arm3_link, child end_short_arm3_link, origin xyz=0 0.075 0
- added joint end_short_arm4_joint: type fixed, parent short_arm4_link, child end_short_arm4_link, origin xyz=0 0.075 0
- added joint end_short_arm5_joint: type fixed, parent short_arm5_link, child end_short_arm5_link, origin xyz=0 0.075 0
- added joint end_short_arm6_joint: type fixed, parent short_arm6_link, child end_short_arm6_link, origin xyz=0 0.075 0
- joint short_arm1_joint: limit lower=-1.5708 upper=1.5708 effort=100 velocity=100 -> lower=-1.5708 upper=1.5708 effort=.12 velocity=5
- joint short_arm2_joint: limit lower=-1.5708 upper=1.5708 effort=100 velocity=100 -> lower=-1.5708 upper=1.5708 effort=.12 velocity=5
- joint short_arm3_joint: limit lower=-1.5708 upper=1.5708 effort=100 velocity=100 -> lower=-1.5708 upper=1.5708 effort=.12 velocity=5
- joint short_arm4_joint: limit lower=-1.5708 upper=1.5708 effort=100 velocity=100 -> lower=-1.5708 upper=1.5708 effort=.12 velocity=5
- joint short_arm5_joint: limit lower=-1.5708 upper=1.5708 effort=100 velocity=100 -> lower=-1.5708 upper=1.5708 effort=.12 velocity=5
- joint short_arm6_joint: limit lower=-1.5708 upper=1.5708 effort=100 velocity=100 -> lower=-1.5708 upper=1.5708 effort=.12 velocity=5

File: urdf/robot.urdf.xacro (robot description, xacro)
@@ -1,6 +1,7 @@
 <?xml version="1.0"?>
 <robot xmlns:xacro="http://www.ros.org/wiki/xacro"  name="robot">
-    <xacro:include filename="robot_base.xacro" />
+    <xacro:include filename="robot_base_2.xacro" />
     <xacro:include filename="robot_arms.xacro" />
+    <xacro:include filename="robot_long_arms.xacro" />
     <xacro:include filename="robot_gazebo.xacro" />
 </robot>

File: urdf/robot_arms.xacro (robot description, xacro)
@@ -1,6 +1,6 @@
 <?xml version="1.0"?>
 <robot xmlns:xacro="http://www.ros.org/wiki/xacro" >
-    <xacro:property name="short_arm_length" value="0.075"/>
-    <xacro:property name="long_arm_length" value="0.190"/>
+    <xacro:property name="short_arm_length" value="0.065"/>
+    <xacro:property name="long_arm_length" value="0.194"/>
     <xacro:macro name="short_arm_link" params="link_name">
         <link name="${link_name}">
@@ -8,5 +8,5 @@
                 <material name="white"/>
                 <geometry>
-                    <cylinder length = "${short_arm_length}" radius = "0.005"/>
+                    <cylinder length = "${short_arm_length}" radius = "0.004"/>
                 </geometry>
                 <origin xyz="0 ${short_arm_length / 2 } 0" rpy="1.5708 0 0"/>
@@ -14,5 +14,5 @@
             <collision>
                 <geometry>
-                    <cylinder length = "${short_arm_length}" radius = "0.005"/>
+                    <cylinder length = "${short_arm_length}" radius = "0.004"/>
                 </geometry>
                 <origin xyz="0 ${short_arm_length / 2 } 0" rpy="1.5708 0 0"/>

File: urdf/robot_gazebo.xacro (robot description, xacro)
@@ -6,4 +6,40 @@
     <!-- Gazebo is unable to use the same <material> tags that are already in the URDF (that RViz uses). -->
     <!-- Instead, we need to add gazebo tags for our links that refer to Gazebo materials -->
+    <gazebo reference="collision_link1">
+        <mu1>0.2</mu1>
+        <mu2>0.3</mu2>
+    </gazebo>
+    <gazebo reference="collision_link2">
+        <mu1>0.2</mu1>
+        <mu2>0.3</mu2>
+    </gazebo>
+    <gazebo reference="collision_link3">
+        <mu1>0.2</mu1>
+        <mu2>0.3</mu2>
+    </gazebo>
+    <gazebo reference="end_short_arm1_link">
+        <mu1>0.2</mu1>
+        <mu2>0.3</mu2>
+    </gazebo>
+    <gazebo reference="end_short_arm2_link">
+        <mu1>0.2</mu1>
+        <mu2>0.3</mu2>
+    </gazebo>
+    <gazebo reference="end_short_arm3_link">
+        <mu1>0.2</mu1>
+        <mu2>0.3</mu2>
+    </gazebo>
+    <gazebo reference="end_short_arm4_link">
+        <mu1>0.2</mu1>
+        <mu2>0.3</mu2>
+    </gazebo>
+    <gazebo reference="end_short_arm5_link">
+        <mu1>0.2</mu1>
+        <mu2>0.3</mu2>
+    </gazebo>
+    <gazebo reference="end_short_arm6_link">
+        <mu1>0.2</mu1>
+        <mu2>0.3</mu2>
+    </gazebo>
     <gazebo reference="base_link">
         <material>Gazebo/Green</material>
@@ -69,5 +105,5 @@
         <plugin name="gazebo_ros_joint_pose_trajectory"
             filename="libgazebo_ros_joint_pose_trajectory.so">
-            <update_rate>20</update_rate>
+            <!--#<update_rate>20</update_rate>-->
         </plugin>
     </gazebo>

File: urdf/robot_long_arms.xacro (robot description, xacro)
@@ -1,183 +1,66 @@
 <?xml version="1.0"?>
 <robot xmlns:xacro="http://www.ros.org/wiki/xacro" >
-    <joint name="long_arm1_joint_x" type="revolute">
-        <parent link="short_arm1_link"/>
-        <child link="long_arm1_link"/>
-        <origin xyz="0 ${short_arm_length} 0" rpy="0 0 0"/>
-        <axis xyz="1 0 0"/>
-        <limit lower="-3" upper="3" effort="100" velocity="100"/>
-    </joint>
-    <link name="long_arm1_link">
-        <visual>
-            <geometry>
-                <sphere radius="0.006"/>
-            </geometry>
-            <origin xyz="0 0 0"/>
-        </visual>
-    </link>
-    <joint name="long_arm1_joint_z" type="revolute">
-        <parent link="long_arm1_link"/>
-        <child link="long_arm1_link2"/>
-        <origin xyz="0 0 0" rpy="0 0 0"/>
-        <axis xyz="0 0 1"/>
-        <limit lower="-3" upper="3" effort="100" velocity="100"/>
-    </joint>
-    <link name="long_arm1_link2">
-        <visual>
-            <geometry>
-                <cylinder length = "${long_arm_length}" radius = "0.003"/>
-            </geometry>
-            <origin xyz="0 ${long_arm_length / 2 } 0" rpy="1.5708 0 0"/>
-        </visual>
-    </link>
-    <joint name="long_arm2_joint_x" type="revolute">
-        <parent link="short_arm2_link"/>
-        <child link="long_arm2_link"/>
-        <origin xyz="0 ${short_arm_length} 0" rpy="0 0 0"/>
-        <axis xyz="1 0 0"/>
-        <limit lower="-3" upper="3" effort="100" velocity="100"/>
-    </joint>
-    <link name="long_arm2_link">
-        <visual>
-            <geometry>
-                <sphere radius="0.006"/>
-            </geometry>
-            <origin xyz="0 0 0"/>
-        </visual>
-    </link>
-    <joint name="long_arm2_joint_z" type="revolute">
-        <parent link="long_arm2_link"/>
-        <child link="long_arm2_link2"/>
-        <origin xyz="0 0 0" rpy="0 0 0"/>
-        <axis xyz="0 0 1"/>
-        <limit lower="-3" upper="3" effort="100" velocity="100"/>
-    </joint>
-    <link name="long_arm2_link2">
-        <visual>
-            <geometry>
-                <cylinder length = "${long_arm_length}" radius = "0.003"/>
-            </geometry>
-            <origin xyz="0 ${long_arm_length / 2 } 0" rpy="1.5708 0 0"/>
-        </visual>
-    </link>
-    <joint name="long_arm3_joint_x" type="revolute">
-        <parent link="short_arm3_link"/>
-        <child link="long_arm3_link"/>
-        <origin xyz="0 ${short_arm_length} 0" rpy="0 0 0"/>
-        <axis xyz="1 0 0"/>
-        <limit lower="-3" upper="3" effort="100" velocity="100"/>
-    </joint>
-    <link name="long_arm3_link">
-        <visual>
-            <geometry>
-                <sphere radius="0.006"/>
-            </geometry>
-            <origin xyz="0 0 0"/>
-        </visual>
-    </link>
-    <joint name="long_arm3_joint_z" type="revolute">
-        <parent link="long_arm3_link"/>
-        <child link="long_arm3_link2"/>
-        <origin xyz="0 0 0" rpy="0 0 0"/>
-        <axis xyz="0 0 1"/>
-        <limit lower="-3" upper="3" effort="100" velocity="100"/>
-    </joint>
-    <link name="long_arm3_link2">
-        <visual>
-            <geometry>
-                <cylinder length = "${long_arm_length}" radius = "0.003"/>
-            </geometry>
-            <origin xyz="0 ${long_arm_length / 2 } 0" rpy="1.5708 0 0"/>
-        </visual>
-    </link>
-    <joint name="long_arm4_joint_x" type="revolute">
-        <parent link="short_arm4_link"/>
-        <child link="long_arm4_link"/>
-        <origin xyz="0 ${short_arm_length} 0" rpy="0 0 0"/>
-        <axis xyz="1 0 0"/>
-        <limit lower="-3" upper="3" effort="100" velocity="100"/>
-    </joint>
-    <link name="long_arm4_link">
-        <visual>
-            <geometry>
-                <sphere radius="0.006"/>
-            </geometry>
-            <origin xyz="0 0 0"/>
-        </visual>
-    </link>
-    <joint name="long_arm4_joint_z" type="revolute">
-        <parent link="long_arm4_link"/>
-        <child link="long_arm4_link2"/>
-        <origin xyz="0 0 0" rpy="0 0 0"/>
-        <axis xyz="0 0 1"/>
-        <limit lower="-3" upper="3" effort="100" velocity="100"/>
-    </joint>
-    <link name="long_arm4_link2">
-        <visual>
-            <geometry>
-                <cylinder length = "${long_arm_length}" radius = "0.003"/>
-            </geometry>
-            <origin xyz="0 ${long_arm_length / 2 } 0" rpy="1.5708 0 0"/>
-        </visual>
-    </link>
-    <joint name="long_arm5_joint_x" type="revolute">
-        <parent link="short_arm5_link"/>
-        <child link="long_arm5_link"/>
-        <origin xyz="0 ${short_arm_length} 0" rpy="0 0 0"/>
-        <axis xyz="1 0 0"/>
-        <limit lower="-3" upper="3" effort="100" velocity="100"/>
-    </joint>
-    <link name="long_arm5_link">
-        <visual>
-            <geometry>
-                <sphere radius="0.006"/>
-            </geometry>
-            <origin xyz="0 0 0"/>
-        </visual>
-    </link>
-    <joint name="long_arm5_joint_z" type="revolute">
-        <parent link="long_arm5_link"/>
-        <child link="long_arm5_link2"/>
-        <origin xyz="0 0 0" rpy="0 0 0"/>
-        <axis xyz="0 0 1"/>
-        <limit lower="-3" upper="3" effort="100" velocity="100"/>
-    </joint>
-    <link name="long_arm5_link2">
-        <visual>
-            <geometry>
-                <cylinder length = "${long_arm_length}" radius = "0.003"/>
-            </geometry>
-            <origin xyz="0 ${long_arm_length / 2 } 0" rpy="1.5708 0 0"/>
-        </visual>
-    </link>
-    <joint name="long_arm6_joint_x" type="revolute">
-        <parent link="short_arm6_link"/>
-        <child link="long_arm6_link"/>
-        <origin xyz="0 ${short_arm_length} 0" rpy="0 0 0"/>
-        <axis xyz="1 0 0"/>
-        <limit lower="-3" upper="3" effort="100" velocity="100"/>
-    </joint>
-    <link name="long_arm6_link">
-        <visual>
-            <geometry>
-                <sphere radius="0.006"/>
-            </geometry>
-            <origin xyz="0 0 0"/>
-        </visual>
-    </link>
-    <joint name="long_arm6_joint_z" type="revolute">
-        <parent link="long_arm6_link"/>
-        <child link="long_arm6_link2"/>
-        <origin xyz="0 0 0" rpy="0 0 0"/>
-        <axis xyz="0 0 1"/>
-        <limit lower="-3" upper="3" effort="100" velocity="100"/>
-    </joint>
-    <link name="long_arm6_link2">
-        <visual>
-            <geometry>
-                <cylinder length = "${long_arm_length}" radius = "0.003"/>
-            </geometry>
-            <origin xyz="0 ${long_arm_length / 2 } 0" rpy="1.5708 0 0"/>
-        </visual>
-    </link>
+    <xacro:property name="short_arm_length" value="0.065"/>
+    <xacro:property name="long_arm_length" value="0.194"/>
+    <xacro:macro name="long_arm" params="number">
+<!--ELBOW JOINT FOR X ROTATION-->
+        <joint name="elbow${number}_x_joint" type="revolute">
+            <parent link="short_arm${number}_link"/>
+            <child link="elbow${number}_link"/>
+            <origin xyz="0 ${short_arm_length} 0" rpy="0 0 0"/>
+            <axis xyz="1 0 0"/>
+            <limit lower="-1.5708" upper="1.5708" effort=".12" velocity="5"/>
+            <dynamics damping="1.0" friction="0.2"/>
+        </joint>
+    <!--ELBOW X LINK-->
+        <link name="elbow${number}_link">
+            <visual>
+                <material name="white"/>
+                <geometry>
+                    <sphere radius="0.005"/>
+                </geometry>
+                <origin xyz="0 0 0" rpy="0 0 0"/>
+            </visual>
+            <inertial>
+                <origin xyz="0 0 0" rpy="0 0 0"/>
+                <mass value="0.060"/>
+                <inertia
+                    ixx="0.00001" ixy="0.0" ixz="0.0"
+                    iyy="0.0000065" iyz="0.0"
+                    izz="0.0000125"/>
+            </inertial>
+        </link>
+    <!--ELBOW Z LINK-->
+        <joint name="elbow${number}_y_joint" type="revolute">
+            <parent link="elbow${number}_link"/>
+            <child link="long_arm${number}_link"/>
+            <origin xyz="0 0 0" rpy="0 0 0"/>
+            <axis xyz="0 0 1"/>
+            <limit lower="-1.5708" upper="1.5708" effort=".12" velocity="5"/>
+            <dynamics damping="1.0" friction="0.2"/>
+        </joint>
+        <link name="long_arm${number}_link">
+            <visual>
+                <material name="white"/>
+                <geometry>
+                    <cylinder length = "${long_arm_length}" radius = "0.0025"/>
+                </geometry>
+                <origin xyz="0 ${long_arm_length / 2 } 0" rpy="1.5708 0 0"/>
+            </visual>
+            <inertial>
+                <origin xyz="0 ${long_arm_length / 2 } 0" rpy="1.5708 0 0"/>
+                <mass value="0.060"/>
+                <inertia
+                    ixx="0.00001" ixy="0.0" ixz="0.0"
+                    iyy="0.0000065" iyz="0.0"
+                    izz="0.0000125"/>
+            </inertial>
+        </link>
+    </xacro:macro>
+    <xacro:long_arm number="1"/>
+    <xacro:long_arm number="2"/>
+    <xacro:long_arm number="3"/>
+    <xacro:long_arm number="4"/>
+    <xacro:long_arm number="5"/>
+    <xacro:long_arm number="6"/>
 </robot>
